Commit message: Refactors r2d2

File: src/my_r2d2/urdf/r2d2.urdf.xacro (robot description, xacro)
@@ -8,4 +8,5 @@
   <xacro:property name="wheeldiam" value="0.07" />
   <xacro:property name="pi" value="3.1415" />
+  <xacro:property name="boxlen" value="0.08" />
   <material name="blue">
     <color rgba="0 0 0.8 1"/>
@@ -23,14 +24,5 @@
     </inertial>
   </xacro:macro>
-  <!-- had to rewrite base_footprint to base, otherwise everything blew up and errored-->
-  <link name="base_footprint">
-    <visual>
-      <geometry>
-        <cylinder radius="${width*2}" length="0.01"/>
-      </geometry>
-      <material name="black"/>
-    </visual>
-  </link>
-  <link name="body_yay">
+  <link name="base_link">
     <visual>
       <geometry>
@@ -46,9 +38,4 @@
     <xacro:default_inertial mass="10"/>
   </link>
-  <joint name="body_yay_to_base_footprint" type="fixed">
-    <parent link="base_footprint"/>
-    <child link="body_yay"/>
-    <origin xyz="0 0 ${bodylen/2+wheeldiam+(wheeldiam/2+.05)}" rpy="0 0 0"/>
-  </joint>
   <xacro:macro name="wheel" params="prefix suffix reflect">
     <link name="${prefix}_${suffix}_wheel">
@@ -81,5 +68,5 @@
           <box size="${leglen} 0.1 0.2"/>
         </geometry>
-        <origin xyz="0 0 ${leglen}" rpy="0 ${pi/2} 0"/>
+        <origin xyz="0 0 -${leglen/2}" rpy="0 ${pi/2} 0"/>
         <material name="white"/>
       </visual>
@@ -88,10 +75,10 @@
           <box size="${leglen} 0.1 0.2"/>
         </geometry>
-        <origin xyz="0 0 0" rpy="0 ${pi/2} 0"/>
+        <origin xyz="0 0 -${leglen/2}" rpy="0 ${pi/2} 0"/>
       </collision>
       <xacro:default_inertial mass="10"/>
     </link>
     <joint name="base_to_${prefix}_leg" type="fixed">
-      <parent link="base_footprint"/>
+      <parent link="base_link"/>
       <child link="${prefix}_leg"/>
       <origin xyz="0 ${reflect*(width+.02)} 0.25" />
@@ -114,5 +101,5 @@
       <parent link="${prefix}_leg"/>
       <child link="${prefix}_base"/>
-      <origin xyz="0 0 0" />
+      <origin xyz="0 0 ${-leglen}" />
     </joint>
     <xacro:wheel prefix="${prefix}" suffix="front" reflect="1"/>
@@ -122,5 +109,5 @@
   <xacro:leg prefix="left" reflect="1" />
   <joint name="gripper_extension" type="prismatic">
-    <parent link="base_footprint"/>
+    <parent link="base_link"/>
     <child link="gripper_pole"/>
     <limit effort="1000.0" lower="-${width*2-.02}" upper="0" velocity="0.5"/>
@@ -202,21 +189,22 @@
   </link>
   <joint name="head_swivel" type="continuous">
-    <parent link="base_footprint"/>
+    <parent link="base_link"/>
     <child link="head"/>
     <axis xyz="0 0 1"/>
-    <origin xyz="0 0 ${bodylen+width}"/>
+    <origin xyz="0 0 ${bodylen/2}"/>
   </joint>
   <link name="box">
     <visual>
       <geometry>
-        <box size="0.08 0.08 0.08"/>
+        <box size="${boxlen} ${boxlen} ${boxlen}"/>
       </geometry>
       <material name="blue"/>
-      <origin xyz="-0.04 0 0"/>
-    </visual>
-    <collision>
-      <geometry>
-        <box size="0.08 0.08 0.08"/>
-      </geometry>
+      <origin xyz="-${boxlen/2} 0 0"/>
+    </visual>
+    <collision>
+      <geometry>
+        <box size="${boxlen} ${boxlen} ${boxlen}"/>
+      </geometry>
+      <origin xyz="-${boxlen/2} 0 0"/>
     </collision>
     <xacro:default_inertial mass="1"/>
@@ -227,24 +215,38 @@
     <origin xyz="${.707*width+0.04} 0 ${.707*width}"/>
   </joint>
-  <link name="lens">
-    <visual>
-      <geometry>
-        <cylinder radius="0.03" length="0.015" />
-      </geometry>
+  <link name="lense">
+    <visual>
+      <geometry>
+        <cylinder length="${boxlen+0.001}" radius="${boxlen/2-0.005}"/>
+      </geometry>
+      <origin rpy="${pi/2} 0 ${pi/2}" xyz="0 0 0"/>
       <material name="black"/>
-      <origin xyz="0 0 0" />
-    </visual>
-    <collision>
-      <geometry>
-        <cylinder radius="0.03" length="0.015" />
-      </geometry>
-      <origin xyz="0 0 0"/>
-    </collision>
-    <xacro:default_inertial mass="1"/>
-  </link>
-  <joint name="lens_to_box" type="fixed">
+    </visual>
+    <collision>
+      <geometry>
+        <cylinder length="${boxlen+0.001}" radius="${boxlen/2-0.005}"/>
+      </geometry>
+      <origin rpy="${pi/2} 0 ${pi/2}" xyz="0 0 0"/>
+    </collision>
+    <xacro:default_inertial mass="0.5"/>
+  </link>
+  <joint name="tolense" type="fixed">
     <parent link="box"/>
-    <child link="lens"/>
-    <origin xyz="0 0 0" rpy="0 ${pi/2} 0"/>
+    <child link="lense"/>
+    <origin xyz="-${boxlen/2} 0 0"/>
+  </joint>
+  <link name="eye">
+  </link>
+  <joint name="toeye" type="fixed">
+    <parent link="lense"/>
+    <child link="eye"/>
+    <origin rpy="-${pi/2} 0 -${pi/2}" xyz="0 0 0"/>
+  </joint>
+  <link name="base_footprint">
+  </link>
+  <joint name="footprint_to_base" type="fixed">
+    <parent link="base_footprint"/>
+    <child link="base_link"/>
+    <origin xyz="0 0 0.47"/>
   </joint>
 </robot>
